File: AltairMD_V3/AltairMD_V3.kicad_pcb (KiCad board)
At the start: 2 copper layers, 0 parts

Commit message: Add files via upload
Parts:
- added C1: 10μ, Capacitor_THT:CP_Radial_D5.0mm_P2.00mm, F.Cu at (138.0, 71.6)
- added C2: 10μ, Capacitor_THT:CP_Radial_D5.0mm_P2.00mm, F.Cu at (138.2, 95.2)
- added C3: 0.1μ, Capacitor_THT:CP_Radial_D5.0mm_P2.00mm, F.Cu at (119.4, 89.0)
- added C4: 0.1μ, Capacitor_THT:CP_Radial_D5.0mm_P2.00mm, F.Cu at (119.4, 99.3)
- added D1: LED, LED_THT:LED_D3.0mm, F.Cu at (99.1, 68.6)
- added D10: LED_Dual_Bidirectional, LED_THT:LED_D3.0mm, F.Cu at (142.2, 116.8)
- added D2: LED, LED_THT:LED_D3.0mm, F.Cu at (92.7, 68.6)
- added D3: LED, LED_THT:LED_D3.0mm, F.Cu at (105.7, 68.6)
- added D4: 1N4148, Diode_THT:D_DO-35_SOD27_P10.16mm_Horizontal, F.Cu at (134.6, 73.7)
- added D5: 1N4148, Diode_THT:D_DO-35_SOD27_P10.16mm_Horizontal, F.Cu at (134.6, 95.2)
- added D6: D_Schottky, Diode_THT:D_DO-35_SOD27_P10.16mm_Horizontal, F.Cu at (167.6, 85.1)
- added D7: D_Schottky, Diode_THT:D_DO-35_SOD27_P10.16mm_Horizontal, F.Cu at (161.8, 97.5)
- added D8: D_Schottky, Diode_THT:D_DO-35_SOD27_P10.16mm_Horizontal, F.Cu at (147.7, 124.6)
- added D9: D_Schottky, Diode_THT:D_DO-35_SOD27_P10.16mm_Horizontal, F.Cu at (123.7, 111.0)
- added J1: Conn_02x20_Odd_Even, Connector_PinHeader_2.54mm:PinHeader_2x20_P2.54mm_Horizontal, F.Cu at (137.2, 121.9)
- added MOSFET1: TK65A10N1, Package_TO_SOT_THT:TO-220-3_Horizontal_TabDown, F.Cu at (159.9, 75.9)
- added MOSFET2: TK65A10N1, Package_TO_SOT_THT:TO-220-3_Horizontal_TabDown, F.Cu at (159.9, 88.9)
- added MOSFET3: TK65A10N1, Package_TO_SOT_THT:TO-220-3_Horizontal_TabDown, F.Cu at (159.9, 101.6)
- added MOSFET4: TK65A10N1, Package_TO_SOT_THT:TO-220-3_Horizontal_TabDown, F.Cu at (159.9, 114.8)
- added R1: 220, Resistor_THT:R_Axial_DIN0207_L6.3mm_D2.5mm_P10.16mm_Horizontal, F.Cu at (99.1, 83.8)
- added R10: Qg 5.25, Resistor_THT:R_Axial_DIN0207_L6.3mm_D2.5mm_P10.16mm_Horizontal, F.Cu at (139.7, 101.6)
- added R11: 10K, Resistor_THT:R_Axial_DIN0207_L6.3mm_D2.5mm_P10.16mm_Horizontal, F.Cu at (139.7, 104.1)
- added R12: Qg, Resistor_THT:R_Axial_DIN0207_L6.3mm_D2.5mm_P10.16mm_Horizontal, F.Cu at (139.7, 106.7)
- added R13: 10K, Resistor_THT:R_Axial_DIN0207_L6.3mm_D2.5mm_P10.16mm_Horizontal, F.Cu at (139.7, 109.2)
- added R14: 550, Resistor_THT:R_Axial_DIN0207_L6.3mm_D2.5mm_P10.16mm_Horizontal, F.Cu at (127.0, 116.8)
- added R2: 220, Resistor_THT:R_Axial_DIN0207_L6.3mm_D2.5mm_P10.16mm_Horizontal, F.Cu at (92.7, 83.8)
- added R3: 1.5k, Resistor_THT:R_Axial_DIN0207_L6.3mm_D2.5mm_P10.16mm_Horizontal, F.Cu at (105.7, 83.8)
- added R4: 220, Resistor_THT:R_Axial_DIN0207_L6.3mm_D2.5mm_P10.16mm_Horizontal, F.Cu at (101.6, 111.5)
- added R5: 220, Resistor_THT:R_Axial_DIN0207_L6.3mm_D2.5mm_P2.54mm_Vertical, F.Cu at (104.1, 100.1)
- added R6: Qg5.25, Resistor_THT:R_Axial_DIN0207_L6.3mm_D2.5mm_P10.16mm_Horizontal, F.Cu at (137.2, 78.7)
- added R7: 10K, Resistor_THT:R_Axial_DIN0207_L6.3mm_D2.5mm_P10.16mm_Horizontal, F.Cu at (137.2, 81.3)
- added R8: Qg, Resistor_THT:R_Axial_DIN0207_L6.3mm_D2.5mm_P10.16mm_Horizontal, F.Cu at (137.2, 86.4)
- added R9: 10K, Resistor_THT:R_Axial_DIN0207_L6.3mm_D2.5mm_P10.16mm_Horizontal, F.Cu at (137.2, 89.2)
- added SW1: SW_DIP_x01, Connector_PinHeader_2.54mm:PinHeader_1x02_P2.54mm_Vertical, F.Cu at (119.6, 108.7)
- added U1: TLP250, Package_DIP:DIP-8_W7.62mm, F.Cu at (106.7, 99.1)
- added U2: TLP250, Package_DIP:DIP-8_W7.62mm, F.Cu at (106.7, 88.9)
- added U3: IR2302, Package_DIP:DIP-8_W7.62mm, F.Cu at (124.5, 78.8)
- added U4: IR2302, Package_DIP:DIP-8_W7.62mm, F.Cu at (126.0, 99.1)
- added U5: 7400, Package_DIP:DIP-14_W7.62mm, F.Cu at (94.0, 94.0)
Routing:
- net GND1: track 0.00 -> 1122.1 mm, vias 0 -> 2
- net M+: track 0.00 -> 403.1 mm, vias 0 -> 2
- net +24V: track 0.00 -> 308.9 mm, vias 0 -> 2
- net M-: track 0.00 -> 278.8 mm
- net +12V: track 0.00 -> 118.1 mm, vias 0 -> 6
- net Net-(U2-Pad2): track 0.00 -> 88.9 mm, vias 0 -> 4
- net +5V: track 0.00 -> 80.4 mm
- net PWM2out: track 0.00 -> 65.3 mm
- net PWM1out: track 0.00 -> 59.4 mm, vias 0 -> 2
- net SD: track 0.00 -> 58.5 mm, vias 0 -> 4
- net PWM: track 0.00 -> 52.1 mm, vias 0 -> 2
- net B: track 0.00 -> 48.5 mm
- net Net-(U1-Pad2): track 0.00 -> 47.4 mm, vias 0 -> 2
- net A: track 0.00 -> 45.2 mm, vias 0 -> 2
- net Net-(MOSFET2-Pad1): track 0.00 -> 20.1 mm
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- added copper zone on B.Cu, net GND1
Other:
- board outline added: 99.8 x 73.7 mm
