File: AltairMD_V3/AltairMD_V3.kicad_sch (KiCad schematic)
At the start: 36 parts, among them J1 Conn_02x20_Odd_Even, U1 TLP250, U2 TLP250, U3 IR2302, U4 IR2302, U5 7400

Commit message: Add files via upload
Parts:
- added C3, C4: 0.1μ, Capacitor_THT:CP_Radial_D5.0mm_P2.00mm, symbol Device:C_Polarized
- added SW1: SW_DIP_x01, Connector_PinHeader_2.54mm:PinHeader_1x02_P2.54mm_Vertical, symbol Switch:SW_DIP_x01
- MOSFET1, MOSFET2, MOSFET3, MOSFET4: footprint (none) -> Package_TO_SOT_THT:TO-220-3_Horizontal_TabDown
- R10: value Qg -> Qg 5.25
- R5: footprint Resistor_THT:R_Axial_DIN0207_L6.3mm_D2.5mm_P10.16mm_Horizontal -> Resistor_THT:R_Axial_DIN0207_L6.3mm_D2.5mm_P2.54mm_Vertical
- R6: value Qg -> Qg5.25
Connections:
- net +12V: now also C3.1, C4.1, SW1.1; no longer D3.2 (A), U3.3 (~{SD}), U4.3 (~{SD})
- net GND1: now also C3.2, C4.2
- net M+: now also J1.1 (Pin_1), J1.3 (Pin_3), J1.5 (Pin_5)
- net M-: now also J1.11 (Pin_11), J1.7 (Pin_7), J1.9 (Pin_9)
- new net SD: D3.2 (A), SW1.2, U3.3 (~{SD}), U4.3 (~{SD})
